File: hardware/BREAD_Slice.kicad_sch (KiCad schematic)
At the start: 15 parts, among them J1 Conn_01x10_Female, J2 I2C_01x04

Commit message: Initial commit
Parts:
- removed C1, C3, C4: 22uF, Capacitor_SMD:C_1206_3216Metric, symbol Device:C_Small
- removed C2: 100nF, Capacitor_SMD:C_1206_3216Metric, symbol Device:C_Small
- removed D1: WS2812B_5050, SparkFun-LED:WS2812-5050-4PIN, symbol SparkFun-LED:WS2812B_5050
- removed HS1: Heatsink_Pad, SparkFun-Fuse:Thermal Pad, symbol Mechanical:Heatsink_Pad
- removed J2: I2C_01x04, Connector_JST:JST_SH_SM04B-SRSS-TB_1x04-1MP_P1.00mm_Horizontal, symbol SparkFun-Connector:I2C_01x04
- removed L1: 4.7uH, Inductor_SMD:L_1210_3225Metric, symbol Device:L_Small
- removed U1: ~, Package_TO_SOT_SMD:TSOT-23-6, symbol SparkFun-DiscreteSemi:AP63205
- added C1, C2: 10uF_t, OCI_UPL_FOOTPRINTS:C_2312, symbol BREAD_Slice-rescue:10uF_t-OCI_UPL_2_Capacitors
- added C10, C11, C12, C13, C14, C3, C4, C5, C6, C7, C8, C9: 1uF_t, OCI_UPL_FOOTPRINTS:C_1206_HandSoldering, symbol BREAD_Slice-rescue:1uF_t-OCI_UPL_2_Capacitors
- added J2, J3, J4, J5: Term_2, OCI_UPL_FOOTPRINTS:TerminalBlock_Pheonix_MKDS1.5-2pol, symbol BREAD_Slice-rescue:Term_2-OCI_UPL_10_Connectors
- added Logo1: Logo_Open_Hardware_Small, Symbol:OSHW-Symbol_6.7x6mm_SilkScreen, symbol Graphic:Logo_Open_Hardware_Small
- added R1, R10, R11, R12, R13, R14, R15, R16, R17, R18, R19, R2, R20, R21, R22, R23, R24, R25, R26, R27, R28, R29, R3, R30, R31, R32, R33, R34, R35, R36, R37, R38, R39, R4, R40, R41, R42, R5, R6, R7, R8, R9: 1K, OCI_UPL_FOOTPRINTS:R_1206_HandSoldering, symbol BREAD_Slice-rescue:1K-OCI_UPL_1_Resistors
- added RV1, RV10, RV11, RV12, RV2, RV3, RV4, RV5, RV6, RV7, RV8, RV9: 10k_t, OCI_UPL_FOOTPRINTS:Potentiometer_Bourns_3296W_3-8Zoll_Inline_ScrewUp, symbol BREAD_Slice-rescue:10k_t-OCI_UPL_1_Resistors
- added U1, U2, U3, U4, U5, U6: MCP6004, Package_DIP:DIP-14_W7.62mm_Socket_LongPads, symbol Amplifier_Operational:MCP6004
- H1, H4: footprint MountingHole:MountingHole_5mm -> MountingHole:MountingHole_3.2mm_M3_DIN965_Pad
- H2: renamed from H3; footprint MountingHole:MountingHole_5mm -> MountingHole:MountingHole_3.2mm_M3_DIN965_Pad
- H3: renamed from H2; footprint MountingHole:MountingHole_5mm -> MountingHole:MountingHole_3.2mm_M3_DIN965_Pad
Connections:
- net +12V: now also A1.30 (VIN), C1.1
- net +5V: now also C2.1, C3.1, C4.1, C5.1, C6.1, C7.1, C8.1, J5.1, RV1.1, RV2.1, RV3.1, RV4.1, RV5.1, RV6.1, U1.4 (V+), U2.4 (V+), U3.4 (V+), U4.4 (V+), U5.4 (V+), U6.4 (V+)
- net GND: now also C1.2, C10.2, C11.2, C12.2, C13.2, C14.2, C2.2, C3.2, C4.2, C5.2, C6.2, C7.2, C8.2, C9.2, J5.2, R19.1, R20.1, R21.1, R22.1, R23.1, R24.1, RV1.3, RV10.3, RV11.3, RV12.3, RV2.3, RV3.3, RV4.3, RV5.3, RV6.3, RV7.3, RV8.3, RV9.3, U1.11 (V-), U2.11 (V-), U3.11 (V-), U4.11 (V-), U5.11 (V-), U6.11 (V-)
- net INT: now also A1.7 (D4), J1.8 (Pin_8); no longer A1.6 (D3), J1.7 (Pin_7)
- net SYNC: now also A1.6 (D3), J1.7 (Pin_7); no longer A1.7 (D4), J1.8 (Pin_8)
- net CH0_AI: now reaches A1.19 (A0)
- net CH0_AI: now also U1.13 (-), U1.14
- net CH1_AI: now reaches A1.20 (A1)
- net CH1_AI: now also U2.13 (-), U2.14
- net CH2_AI: now reaches A1.21 (A2)
- net CH2_AI: now also U3.13 (-), U3.14
- net CH3_AI: now reaches A1.22 (A3)
- net CH3_AI: now also U4.13 (-), U4.14
- net CH4_AI: now reaches A1.25 (A6)
- net CH4_AI: now also U5.13 (-), U5.14
- net CH5_AI: now reaches A1.26 (A7)
- net CH5_AI: now also U6.13 (-), U6.14
- net LED: no longer names the net of A1.8 (D5)
- new net: R1.2, R8.1, U1.1
- new net: R1.1, U1.2 (-)
- new net: RV1.2, U1.3 (+)
- new net: R19.2, R7.2, U1.5 (+)
- new net: R25.1, R8.2, U1.6 (-)
- new net: R25.2, U1.10 (+), U1.7
- new net: R37.1, RV7.1, U1.8
- new net: R31.1, U1.9 (-)
- new net: C9.1, R37.2, U1.12 (+)
- new net: R31.2, RV7.2
- new net: R10.1, R2.2, U2.1
- new net: R2.1, U2.2 (-)
- new net: RV2.2, U2.3 (+)
- new net: R20.2, R9.2, U2.5 (+)
- new net: R10.2, R26.1, U2.6 (-)
- new net: R26.2, U2.10 (+), U2.7
- new net: R38.1, RV8.1, U2.8
- new net: R32.1, U2.9 (-)
- new net: C10.1, R38.2, U2.12 (+)
- new net: R32.2, RV8.2
- new net: R12.1, R3.2, U3.1
- new net: R3.1, U3.2 (-)
- new net: RV3.2, U3.3 (+)
- new net: R11.2, R21.2, U3.5 (+)
- new net: R12.2, R27.1, U3.6 (-)
- new net: R27.2, U3.10 (+), U3.7
- new net: R39.1, RV9.1, U3.8
- new net: R33.1, U3.9 (-)
- new net: C11.1, R39.2, U3.12 (+)
- new net: R33.2, RV9.2
- new net: R14.1, R4.2, U4.1
- new net: R4.1, U4.2 (-)
- new net: RV4.2, U4.3 (+)
- new net: R13.2, R22.2, U4.5 (+)
- new net: R14.2, R28.1, U4.6 (-)
- new net: R28.2, U4.10 (+), U4.7
- new net: R40.1, RV10.1, U4.8
- new net: R34.1, U4.9 (-)
- new net: C12.1, R40.2, U4.12 (+)
- new net: R34.2, RV10.2
- new net: R16.1, R5.2, U5.1
- new net: R5.1, U5.2 (-)
- new net: RV5.2, U5.3 (+)
- new net: R15.2, R23.2, U5.5 (+)
- new net: R16.2, R29.1, U5.6 (-)
- new net: R29.2, U5.10 (+), U5.7
- new net: R41.1, RV11.1, U5.8
- new net: R35.1, U5.9 (-)
- new net: C13.1, R41.2, U5.12 (+)
- new net: R35.2, RV11.2
- new net: R18.1, R6.2, U6.1
- new net: R6.1, U6.2 (-)
- new net: RV6.2, U6.3 (+)
- new net: R17.2, R24.2, U6.5 (+)
- new net: R18.2, R30.1, U6.6 (-)
- new net: R30.2, U6.10 (+), U6.7
- new net: R42.1, RV12.1, U6.8
- new net: R36.1, U6.9 (-)
- new net: C14.1, R42.2, U6.12 (+)
- new net: R36.2, RV12.2
- new net Ch0_in: J2.1, R7.1
- new net Ch1_in: J2.2, R9.1
- new net Ch2_in: J3.1, R11.1
- new net Ch3_in: J3.2, R13.1
- new net Ch4_in: J4.1, R15.1
- new net Ch5_in: J4.2, R17.1
- no-connect marks 22 -> 15
Other:
- moved on the sheet: A1, H1, H2, H3, H4, J1

Commit message: extensive documentation, remade board, subcircuits for all
Parts:
- removed C1, C2: 10uF_t, OCI_UPL_FOOTPRINTS:C_2312, symbol BREAD_Slice-rescue:10uF_t-OCI_UPL_2_Capacitors
- removed C10, C11, C12, C13, C14, C3, C4, C5, C6, C7, C8, C9: 1uF_t, OCI_UPL_FOOTPRINTS:C_1206_HandSoldering, symbol BREAD_Slice-rescue:1uF_t-OCI_UPL_2_Capacitors
- removed J2: Term_2, OCI_UPL_FOOTPRINTS:TerminalBlock_Pheonix_MKDS1.5-2pol, symbol BREAD_Slice-rescue:Term_2-OCI_UPL_10_Connectors
- removed Logo1: Logo_Open_Hardware_Small, Symbol:OSHW-Symbol_6.7x6mm_SilkScreen, symbol Graphic:Logo_Open_Hardware_Small
- removed R1, R10, R11, R12, R13, R14, R15, R16, R17, R18, R19, R2, R20, R21, R22, R23, R24, R25, R26, R27, R28, R29, R3, R30, R31, R32, R33, R34, R35, R36, R37, R38, R39, R4, R40, R41, R42, R5, R6, R7, R8, R9: 1K, OCI_UPL_FOOTPRINTS:R_1206_HandSoldering, symbol BREAD_Slice-rescue:1K-OCI_UPL_1_Resistors
- removed RV1, RV10, RV11, RV12, RV2, RV3, RV4, RV5, RV6, RV7, RV8, RV9: 10k_t, OCI_UPL_FOOTPRINTS:Potentiometer_Bourns_3296W_3-8Zoll_Inline_ScrewUp, symbol BREAD_Slice-rescue:10k_t-OCI_UPL_1_Resistors
- removed U1, U2, U3, U4, U5, U6: MCP6004, Package_DIP:DIP-14_W7.62mm_Socket_LongPads, symbol Amplifier_Operational:MCP6004
- added C1, C3, C4: 22uF, Capacitor_SMD:C_1206_3216Metric, symbol Device:C_Small
- added C2: 100nF, Capacitor_SMD:C_1206_3216Metric, symbol Device:C_Small
- added D1: WS2812B_5050, SparkFun-LED:WS2812-5050-4PIN, symbol SparkFun-LED:WS2812B_5050
- added HS1: Heatsink_Pad, KML-Custom:Thermal Pad, symbol Mechanical:Heatsink_Pad
- added J1: I2C_01x04, Connector_JST:JST_SH_SM04B-SRSS-TB_1x04-1MP_P1.00mm_Horizontal, symbol SparkFun-Connector:I2C_01x04
- added J6, J7, J8: Term_2, TerminalBlock_Phoenix:TerminalBlock_Phoenix_MKDS-1,5-2_1x02_P5.00mm_Horizontal, symbol BREAD_Slice-rescue:Term_2-OCI_UPL_10_Connectors
- added L1: 4.7uH, Inductor_SMD:L_1210_3225Metric, symbol Device:L_Small
- added U1: ~, Package_TO_SOT_SMD:TSOT-23-6, symbol SparkFun-DiscreteSemi:AP63205
- H1, H4: footprint MountingHole:MountingHole_3.2mm_M3_DIN965_Pad -> MountingHole:MountingHole_5mm
- H2: renamed from H3; footprint MountingHole:MountingHole_3.2mm_M3_DIN965_Pad -> MountingHole:MountingHole_5mm
- H3: renamed from H2; footprint MountingHole:MountingHole_3.2mm_M3_DIN965_Pad -> MountingHole:MountingHole_5mm
- J3, J4, J5: footprint OCI_UPL_FOOTPRINTS:TerminalBlock_Pheonix_MKDS1.5-2pol -> TerminalBlock_Phoenix:TerminalBlock_Phoenix_MKDS-1,5-2_1x02_P5.00mm_Horizontal
- renumbered J1 to J2
Connections:
- net +12V: now also C1.2, U1.2 (EN), U1.3 (VIN); no longer A1.30 (VIN)
- net +5V: now also C3.2, C4.2, D1.1 (VDD), J1.2 (Pin_2), J6.1, J7.1, J8.1, L1.2, U1.1 (FB); no longer J5.1
- net CH0_AI: now also A1.22 (A3); no longer A1.19 (A0)
- net CH1_AI: now also A1.25 (A6); no longer A1.20 (A1)
- net CH3_AI: now also A1.26 (A7); no longer A1.22 (A3)
- net CH4_AI: now also A1.20 (A1); no longer A1.25 (A6)
- net CH5_AI: now also A1.19 (A0); no longer A1.26 (A7)
- net Ch0_in: now also J3.1
- net Ch1_in: now also J3.2
- net Ch2_in: now also J4.1; no longer J3.1
- net Ch3_in: now also J4.2; no longer J3.2
- net Ch4_in: now also J5.1; no longer J4.1
- net Ch5_in: now also J5.2; no longer J4.2
- net GND: now also C1.1, C3.1, C4.1, D1.3 (VSS), HS1.1, J1.1 (Pin_1), J6.2, J7.2, J8.2, U1.4 (GND); no longer J5.2
- net I2C_CLK: now also J1.4 (Pin_4)
- net I2C_DAT: now also J1.3 (Pin_3)
- net INT: now also A1.6 (D3), J2.7 (Pin_7); no longer A1.7 (D4), J2.8 (Pin_8)
- net SYNC: now also A1.7 (D4), J2.8 (Pin_8); no longer A1.6 (D3), J2.7 (Pin_7)
- net LED: now reaches A1.8 (D5)
- net LED: now also D1.4 (DIN)
- new net: C2.1, L1.1, U1.5 (SW)
- new net: C2.2, U1.6 (BST)
- no-connect marks 15 -> 16
Other:
- added sheet Low Voltage Analog Input (lvai.kicad_sch)
- added sheet Low Voltage Analog Input1 (lvai.kicad_sch)
- added sheet Low Voltage Analog Input2 (lvai.kicad_sch)
- added sheet Low Voltage Analog Input3 (lvai.kicad_sch)
- added sheet Low Voltage Analog Input4 (lvai.kicad_sch)
- added sheet Low Voltage Analog Input5 (lvai.kicad_sch)
- moved on the sheet: A1, H1, H2, H3, H4, J2
